File: 6502 Dev Board.sch (KiCad schematic (older format))
At the start: 36 parts, among them J1 Barrel_Jack, J2 Signals, J3 Addresses, J4 Data, SW1 Power, SW2 Reset, U1 W65C02S, U2 62256, U3 L7805, U4 DS1233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

Commit message: Update metadata.
Other:
- moved on the sheet: C1, C2, C3, C4, C5, C6, C7, C8, D1, D2, D3, D4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
